Commit message: removed franka_hand and gripper. TCP set to last link
Signed-off-by: Iván López Broceño <ivanlpzbrc01@gmail.com>

File: urdf/panda_calibrated_left.urdf (robot description, URDF)
Before this commit: robot panda_left, 14 links, 13 joints
Links:
- removed link ball_left_link
- removed link panda_left_hand
- removed link panda_left_hand_tcp
- removed link panda_left_leftfinger
- removed link panda_left_rightfinger
Joints:
- removed joint ball_left_joint
- removed joint panda_left_finger_joint1
- removed joint panda_left_finger_joint2
- removed joint panda_left_hand_joint
- removed joint panda_left_hand_tcp_joint

File: urdf/panda_calibrated_right.urdf (robot description, URDF)
Before this commit: robot panda_right, 14 links, 13 joints
Links:
- removed link ball_right_link
- removed link panda_right_hand
- removed link panda_right_hand_tcp
- removed link panda_right_leftfinger
- removed link panda_right_rightfinger
Joints:
- removed joint ball_right_joint
- removed joint panda_right_finger_joint1
- removed joint panda_right_finger_joint2
- removed joint panda_right_hand_joint
- removed joint panda_right_hand_tcp_joint
